Commit message: update urdf

File: urdf/servingrobot.urdf (robot description, URDF)
Before this commit: robot servingrobot, 5 links, 4 joints
Links:
- added link base_footprint; visual box size=0.001 0.001 0.001
Joints:
- added joint base_link_joint: type fixed, parent base_footprint, child base_link, origin xyz=0 0 ${wheel_radius + 0.8} rpy=0 0 0

Commit message: t

File: urdf/servingrobot.urdf (robot description, URDF)
Before this commit: robot servingrobot, 6 links, 5 joints
Links:
- added link imu_link; visual box size=0.001 0.001 0.001
Joints:
- added joint imu_link_joint: type fixed, parent base_link, child imu_link, origin xyz=0 0 -0.5 rpy=0 0 0, axis 0 0 1
